Commit message: qqqqq

File: car_description/auonomous_description/urdf/auonomous_description.xacro (robot description, xacro)
@@ -298,4 +298,6 @@
     </collision>
   </link>
+   <link name="laser">
+    </link>
   <joint
     name="lidar_Link_joint"

Commit message: laser

File: car_description/auonomous_description/urdf/auonomous_description.xacro (robot description, xacro)
@@ -298,6 +298,4 @@
     </collision>
   </link>
-   <link name="laser">
-    </link>
   <joint
     name="lidar_Link_joint"
